File: PCB/SPARC-backups/SPARC-2023-03-03_171640/SPARC.kicad_sch (KiCad schematic)
At the start: 86 parts, among them J1 Conn_Coaxial_Power, J2 Conn_Coaxial_Power, J3 Conn_01x06_Female, J4 Conn_01x03_Female, J5 Conn_01x03_Female, J6 Conn_01x06_Female, U1 HV2621, U2 HV2621

Commit message: Changed resistors and added jumpers
Parts:
- JP2, JP3: footprint Connector_PinHeader_2.54mm:PinHeader_1x03_P2.54mm_Vertical -> (none)
Connections:
- net DIN_1: no longer JP2.1 (A)
- net DOUT_0: no longer JP2.3 (B)
- new net Din_1: JP2.1 (A)
- new net Dout_0: JP2.3 (B)
Changed lines of the file:
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@@
     (effects (font (size 1.27 1.27)) (justify left bottom))
   )
-  (label "DIN_1" (at 112.395 196.215 0)
+  (label "Din_1" (at 112.395 196.215 0)
     (effects (font (size 1.27 1.27)) (justify left bottom))
   )
@@
     (effects (font (size 1.27 1.27)) (justify left bottom))
   )
-  (label "DOUT_0" (at 99.695 195.834 0)
+  (label "Dout_0" (at 99.695 195.834 0)
     (effects (font (size 1.27 1.27)) (justify left bottom))
   )
@@
     (property "Reference" "JP3" (id 0) (at 144.907 187.833 0))
     (property "Value" "Jumper_3_Open" (id 1) (at 144.907 190.373 0))
-    (property "Footprint" "Connector_PinHeader_2.54mm:PinHeader_1x03_P2.54mm_Vertical" (id 2) (at 135.128 192.151 0)
+    (property "Footprint" "" (id 2) (at 135.128 192.151 0)
       (effects (font (size 1.27 1.27)) hide)
     )
@@
     (property "Reference" "JP2" (id 0) (at 115.824 187.706 0))
     (property "Value" "Jumper_3_Open" (id 1) (at 115.824 190.246 0))
-    (property "Footprint" "Connector_PinHeader_2.54mm:PinHeader_1x03_P2.54mm_Vertical" (id 2) (at 106.045 192.024 0)
+    (property "Footprint" "" (id 2) (at 106.045 192.024 0)
       (effects (font (size 1.27 1.27)) hide)
     )
@@
     )
     (path "/42e48dc9-76bd-4fd9-8b63-b8544920c97d"
-      (reference "JP2") (unit 1) (value "Jumper_3_Open") (footprint "Connector_PinHeader_2.54mm:PinHeader_1x03_P2.54mm_Vertical")
+      (reference "JP2") (unit 1) (value "Jumper_3_Open") (footprint "")
     )
     (path "/3bcb879b-e5d7-4f89-ab71-b17ebf79b2ae"
-      (reference "JP3") (unit 1) (value "Jumper_3_Open") (footprint "Connector_PinHeader_2.54mm:PinHeader_1x03_P2.54mm_Vertical")
+      (reference "JP3") (unit 1) (value "Jumper_3_Open") (footprint "")
     )
     (path "/29dd5ee0-d7e3-489b-b772-f518721d85c0"
